File: DJet ECU Tester/PCB/DJetECUTester/USBandPower.sch (KiCad schematic (older format))
At the start: 16 parts, among them J3 USB_B_Mini, U2 LM2596S-5, U3 FT232RL

Commit message: Working on new schematic diagram.
Parts:
- J3: symbol Connector:USB_B_Mini -> DJetECUTester-rescue:USB_B_Mini-Connector
Changed lines of the file:
@@
 $Descr A4 11693 8268
 encoding utf-8
-Sheet 2 7
+Sheet 2 6
 Title "D-Jetronic ECU Tester"
-Date "2021-04-04"
-Rev "1.1"
-Comp "(C) Britishideas 2021"
+Date "2022-09-17"
+Rev "2.0"
+Comp "(C) Britishideas 2021-2022"
 Comment1 ""
 Comment2 ""
@@
 	3150 2350 3150 2450
 $Comp
-L Connector:USB_B_Mini J?
+L DJetECUTester-rescue:USB_B_Mini-Connector J?
 U 1 1 6049775F
 P 2450 3200
