File: DJet ECU Tester/PCB/DJetECUTester/Temperature.sch (KiCad schematic (older format))
At the start: 14 parts, among them U4 MCP41HV51-502E-ST, U5 MCP41HV51-502E-ST

Commit message: Added IO multiplexer. Working on additional coolant temperature options. Added status LED back in.
Parts:
- added R?: 7k, Resistor_SMD:R_0805_2012Metric, symbol Device:R
- added R?: 25k, Resistor_SMD:R_0805_2012Metric, symbol Device:R
Connections:
- net ECU_COOLANTTEMP: no longer JP3.2 (Pin_2)
- new net R_BASED_CTEMP: JP3.2 (Pin_2)
Other:
- note added: "7k = 25.21F\n25k = -20.76F"
- moved on the sheet: C14, C15, C16, C17, JP2, JP3, R15, R16, TP1, TP2, TP3, TP4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

Commit message: Completed new schematic.
Parts:
- removed R?: 7k, Resistor_SMD:R_0805_2012Metric, symbol Device:R
- removed R?: 25k, Resistor_SMD:R_0805_2012Metric, symbol Device:R
- added C19, C20: 100nF, Capacitor_SMD:C_0805_2012Metric, symbol Device:C
- added JP1: COOLANTTEMP, Connector_PinHeader_2.54mm:PinHeader_2x01_P2.54mm_Vertical, symbol Connector_Generic:Conn_01x02
- added R45: 100k, Resistor_SMD:R_0805_2012Metric, symbol Device:R
- added TP10, TP11: TestPoint, TestPoint:TestPoint_Pad_D2.0mm, symbol Connector:TestPoint
- added U7: MCP41HV51-502E-ST, Package_SO:TSSOP-14_4.4x5mm_P0.65mm, symbol BritishIdeas:MCP41HV51-502E-ST
- U4, U5: manf2# (none) -> MCP41HV31-502E/ST
Connections:
- net R_BASED_CTEMP is gone; now on net ECU_COOLANTTEMP: JP3.2 (Pin_2)
- net +12V: now also C20.1, U7.14 (V+)
- net +5V: now also C19.1, R45.1, U7.1 (VL), U7.7 (~SHDN)
- net GND: now also C19.2, C20.2, TP11.1, U7.10 (V-), U7.11 (P0B), U7.6 (~WLAT), U7.9 (DGND); no longer TP4.1, U5.11 (P0B)
- net MISO: now also U7.5 (SDO)
- net MOSI: now also U7.4 (SDI)
- net SCK: now also U7.2 (SCK)
- net ~COOLANTTEMP_CS renamed ~COOLANTTEMP1_CS
- new net: JP1.1 (Pin_1), TP4.1, U5.11 (P0B)
- new net: JP1.2 (Pin_2), TP10.1, U7.12 (P0W)
- new net ~COOLANTTEMP2_CS: R45.2, U7.3 (~CS)
- no-connect marks 2 -> 3
Other:
- note removed: "7k = 25.21F\n25k = -20.76F"
- moved on the sheet: C15, C17

Commit message: Updated symbols from rescue to library.
Parts:
- U4, U5, U7: symbol BritishIdeas:MCP41HV51-502E-ST -> DJetECUTester-rescue:MCP41HV51-502E-ST-BritishIdeas
Changed lines of the file:
@@
 $EndComp
 $Comp
-L BritishIdeas:MCP41HV51-502E-ST U4
+L DJetECUTester-rescue:MCP41HV51-502E-ST-BritishIdeas U4
 U 1 1 6045CA2E
 P 4150 2200
@@
 $EndComp
 $Comp
-L BritishIdeas:MCP41HV51-502E-ST U5
+L DJetECUTester-rescue:MCP41HV51-502E-ST-BritishIdeas U5
 U 1 1 60474591
 P 4150 4500
@@
 $EndComp
 $Comp
-L BritishIdeas:MCP41HV51-502E-ST U7
+L DJetECUTester-rescue:MCP41HV51-502E-ST-BritishIdeas U7
 U 1 1 632D874D
 P 4150 6450
